File: schematics/kiCad/blinky-cube.kicad_pcb (KiCad board)
At the start: 2 copper layers, 86.4 x 48.3 mm, 16 parts, among them J2 Barrel_Jack_Switch, J4 Screw_Terminal_01x02, J5 Screw_Terminal_01x02, SW1 SW_Push, U1 Pico, U2 LM4040LP-3

Commit message: added logo
Parts:
- added G***: LOGO, blinkyLiteLogo:blinkyLiteLogo, F.Cu at (136.5, 100.3)
Other:
- board text added: "blinky-adc-v1"
